Commit message: chore: refresh fr3_compare_bundle after union-volume fixes

File: assets/fr3_compare_bundle/fr3_convex.urdf (robot description, URDF)
Before this commit: robot bot, 14 links, 13 joints
Links:
- link fr3_link1: geometry collision mesh filename=meshes/link1_2.obj; visual mesh filename=meshes/link1.dae
- link fr3_link2: geometry collision mesh filename=meshes/link2_2.obj; visual mesh filename=meshes/link2.dae
- link fr3_link3: geometry collision mesh filename=meshes/link3_2.obj; visual mesh filename=meshes/link3.dae
- link fr3_link4: geometry collision mesh filename=meshes/link4_2.obj; visual mesh filename=meshes/link4.dae
- link fr3_link5: geometry collision mesh filename=meshes/link5_2.obj; visual mesh filename=meshes/link5.dae
- link fr3_link6: geometry collision mesh filename=meshes/link6_2.obj; visual mesh filename=meshes/link6.dae
- link fr3_link7: geometry collision mesh filename=meshes/link7_2.obj; visual mesh filename=meshes/link7.dae
- link hand_hand: geometry collision mesh filename=meshes/hand_2.obj; visual mesh filename=meshes/hand.dae
- link hand_leftfinger: geometry collision mesh filename=meshes/flex_griper_connect_2.obj; visual mesh filename=meshes/flex_griper_connect.stl
- link hand_rightfinger: geometry collision mesh filename=meshes/flex_griper_connect_2.obj; visual mesh filename=meshes/flex_griper_connect.stl

File: assets/fr3_compare_bundle/fr3_sphere_default.urdf (robot description, URDF)
Before this commit: robot bot, 14 links, 13 joints
Links:
- link fr3_link0: geometry collision sphere radius=0.019236; collision sphere radius=0.026175
- link fr3_link1: geometry collision sphere radius=0.016680; collision sphere radius=0.031338
- link fr3_link2: geometry collision sphere radius=0.032312; collision sphere radius=0.034652
- link fr3_link3: geometry collision sphere radius=0.029829; collision sphere radius=0.038257
- link fr3_link4: geometry collision sphere radius=0.029371; collision sphere radius=0.034599
- link fr3_link5: geometry collision sphere radius=0.036017; collision sphere radius=0.037193
- link fr3_link6: geometry collision sphere radius=0.032942; collision sphere radius=0.038000
- link fr3_link7: geometry collision sphere radius=0.019873; collision sphere radius=0.020777
- link hand_hand: geometry collision sphere radius=0.029047; collision sphere radius=0.034280
- link hand_leftfinger: geometry collision sphere radius=0.009485; collision sphere radius=0.010171
- link hand_rightfinger: geometry collision sphere radius=0.013646; collision sphere radius=0.014128

File: assets/fr3_compare_bundle/fr3_sphere_single.urdf (robot description, URDF)
Before this commit: robot bot, 14 links, 13 joints
Links:
- link fr3_link0: geometry collision sphere radius=0.128194; visual mesh filename=meshes/link0.dae
- link fr3_link1: geometry collision sphere radius=0.144061; visual mesh filename=meshes/link1.dae
- link fr3_link2: geometry collision sphere radius=0.144440; visual mesh filename=meshes/link2.dae
- link fr3_link3: geometry collision sphere radius=0.128203; visual mesh filename=meshes/link3.dae
- link fr3_link4: geometry collision sphere radius=0.127993; visual mesh filename=meshes/link4.dae
- link fr3_link5: geometry collision sphere radius=0.174640; visual mesh filename=meshes/link5.dae
- link fr3_link6: geometry collision sphere radius=0.098549; visual mesh filename=meshes/link6.dae
- link fr3_link7: geometry collision sphere radius=0.073167; visual mesh filename=meshes/link7.dae
- link hand_hand: geometry collision sphere radius=0.107174; visual mesh filename=meshes/hand.dae
- link hand_rightfinger: geometry collision sphere radius=0.064490; visual mesh filename=meshes/flex_griper_connect.stl

Commit message: fix: include JSON sidecars in compare-all bundle
_run_compare() now copies each variant's JSON sidecar into the
bundle directory alongside the URDF. Previously only URDFs and
meshes were bundled; the analytic capsule/sphere parameters are
now available for inspection.

File: assets/fr3_compare_bundle/fr3_convex.urdf (robot description, URDF)
Before this commit: robot bot, 14 links, 13 joints
Links:
- link fr3_link0: geometry collision mesh filename=meshes/link0_2.obj; visual mesh filename=meshes/link0.dae
- link fr3_link1: geometry collision mesh filename=meshes/link1_3.obj; visual mesh filename=meshes/link1.dae
- link fr3_link2: geometry collision mesh filename=meshes/link2_3.obj; visual mesh filename=meshes/link2.dae
- link fr3_link3: geometry collision mesh filename=meshes/link3_3.obj; visual mesh filename=meshes/link3.dae
- link fr3_link5: geometry collision mesh filename=meshes/link5_3.obj; visual mesh filename=meshes/link5.dae
- link hand_hand: geometry collision mesh filename=meshes/hand_3.obj; visual mesh filename=meshes/hand.dae

File: assets/fr3_compare_bundle/fr3_sphere_default.urdf (robot description, URDF)
Before this commit: robot bot, 14 links, 13 joints
Links:
- link fr3_link0: geometry collision sphere radius=0.017509; collision sphere radius=0.026166
- link fr3_link1: geometry collision sphere radius=0.022111; collision sphere radius=0.044285
- link fr3_link2: geometry collision sphere radius=0.042006; collision sphere radius=0.046565
- link fr3_link3: geometry collision sphere radius=0.026748; collision sphere radius=0.031446
- link fr3_link4: geometry collision sphere radius=0.007279; collision sphere radius=0.032416
- link fr3_link5: geometry collision sphere radius=0.039338; collision sphere radius=0.039793
- link fr3_link6: geometry collision sphere radius=0.036975; collision sphere radius=0.041978
- link fr3_link7: geometry collision sphere radius=0.022339; collision sphere radius=0.024453
- link hand_hand: geometry collision sphere radius=0.028756; collision sphere radius=0.028885
- link hand_leftfinger: geometry collision sphere radius=0.013462; collision sphere radius=0.014401
- link hand_rightfinger: geometry collision sphere radius=0.013164; collision sphere radius=0.015019

File: assets/fr3_compare_bundle/fr3_sphere_single.urdf (robot description, URDF)
Before this commit: robot bot, 14 links, 13 joints
Links:
- link fr3_link0: geometry collision sphere radius=0.128537; visual mesh filename=meshes/link0.dae
- link fr3_link1: geometry collision sphere radius=0.143918; visual mesh filename=meshes/link1.dae
- link fr3_link2: geometry collision sphere radius=0.143744; visual mesh filename=meshes/link2.dae
- link fr3_link3: geometry collision sphere radius=0.128239; visual mesh filename=meshes/link3.dae
- link fr3_link4: geometry collision sphere radius=0.128380; visual mesh filename=meshes/link4.dae
- link fr3_link5: geometry collision sphere radius=0.173660; visual mesh filename=meshes/link5.dae
- link fr3_link6: geometry collision sphere radius=0.098768; visual mesh filename=meshes/link6.dae
- link fr3_link7: geometry collision sphere radius=0.072953; visual mesh filename=meshes/link7.dae
- link hand_hand: geometry collision sphere radius=0.108313; visual mesh filename=meshes/hand.dae
- link hand_rightfinger: geometry collision sphere radius=0.064357; visual mesh filename=meshes/flex_griper_connect.stl
