Commit message: fix: reviewer corrections — paths, wording, verification record
- Fix absolute paths in synthetic URDF files to relative (../meshes/)
- Fix absolute path in fig-capsule-method-schematic RESULT.md
- Replace 'perfect surface coverage' with sampling-qualified language
- Replace 'conservative collision estimates' with 'inner (under-approximating)'
- Add Observed Results table to final verification record

File: doc/paper/artifacts/synthetic-morphology-benchmark/urdf/elbow_tube.urdf (robot description, URDF)
Before this commit: robot elbow_tube, 2 links, 1 joints
Links:
- link elbow_tube: geometry collision mesh filename=../meshes/elbow_tube.obj scale=1 1 1; visual mesh filename=../meshes/elbow_tube.obj scale=1 1 1

File: doc/paper/artifacts/synthetic-morphology-benchmark/urdf/flat_plate.urdf (robot description, URDF)
Before this commit: robot flat_plate, 2 links, 1 joints
Links:
- link flat_plate: geometry collision mesh filename=../meshes/flat_plate.obj scale=1 1 1; visual mesh filename=../meshes/flat_plate.obj scale=1 1 1

File: doc/paper/artifacts/synthetic-morphology-benchmark/urdf/straight_tube.urdf (robot description, URDF)
Before this commit: robot straight_tube, 2 links, 1 joints
Links:
- link straight_tube: geometry collision mesh filename=../meshes/straight_tube.obj scale=1 1 1; visual mesh filename=../meshes/straight_tube.obj scale=1 1 1

File: doc/paper/artifacts/synthetic-morphology-benchmark/urdf/t_branch.urdf (robot description, URDF)
Before this commit: robot t_branch, 2 links, 1 joints
Links:
- link t_branch: geometry collision mesh filename=../meshes/t_branch.obj scale=1 1 1; visual mesh filename=../meshes/t_branch.obj scale=1 1 1

File: doc/paper/artifacts/synthetic-morphology-benchmark/urdf/tapered_tube.urdf (robot description, URDF)
Before this commit: robot tapered_tube, 2 links, 1 joints
Links:
- link tapered_tube: geometry collision mesh filename=../meshes/tapered_tube.obj scale=1 1 1; visual mesh filename=../meshes/tapered_tube.obj scale=1 1 1
